File: Elektronik/Raspberry-Motorsteuerung/raspberrypi_hat.kicad_pcb (KiCad board)
At the start: 4 copper layers, 65 x 56 mm, 20 parts, among them J1 Barrel_Jack_Switch, J2 M04JST-PTH, J3 40HAT, J9 CONN_01X02, Q1 DMG2305UX, Q2 DMMT5401, U2 CAT24C32, U3 R-78E5.0-1.0

Commit message: finished schema, started pcb
Parts:
- added D1: LED, LED_THT:LED_D5.0mm, F.Cu at (81.3, 87.6)
- added D2: LED, LED_THT:LED_D5.0mm, F.Cu at (81.3, 102.9)
- added D3: LED, LED_THT:LED_D5.0mm, F.Cu at (81.3, 95.2)
- added J10: Conn_01x02_Male, Connector_JST:JST_EH_S2B-EH_1x02_P2.50mm_Horizontal, F.Cu at (132.1, 110.5)
- added J11: Conn_01x02_Male, Connector_JST:JST_EH_S2B-EH_1x02_P2.50mm_Horizontal, F.Cu at (109.2, 110.5)
- added J15: Conn_01x02_Male, Connector_JST:JST_EH_S2B-EH_1x02_P2.50mm_Horizontal, F.Cu at (100.3, 110.5)
- added J6: Conn_01x04_Male, Connector_JST:JST_EH_S4B-EH_1x04_P2.50mm_Horizontal, F.Cu at (137.2, 71.1)
- added J8: Conn_01x02_Male, Connector_JST:JST_EH_S2B-EH_1x02_P2.50mm_Horizontal, F.Cu at (91.4, 110.5)
- added R1: 5K, Resistor_SMD:R_0603_1608Metric_Pad0.98x0.95mm_HandSolder, F.Cu at (82.5, 81.3)
- added R2: 5K, Resistor_SMD:R_0603_1608Metric_Pad0.98x0.95mm_HandSolder, F.Cu at (85.1, 81.3)
- added R3: 5K, Resistor_SMD:R_0603_1608Metric_Pad0.98x0.95mm_HandSolder, F.Cu at (80.0, 81.3)
- C1: moved to B.Cu
- J2: value M04JST-PTH -> Conn_01x04_Male; footprint JST-4-PTH -> Connector_JST:JST_EH_S4B-EH_1x04_P2.50mm_Horizontal
- moved J1 65.3 mm to (147.3, 101.6), turned to 90 degrees
- moved U3 21.7 mm to (101.6, 74.9)
- moved A1 20.6 mm to (110.5, 99.1), turned to 90 degrees
- moved J2 19.3 mm to (123.2, 110.5), turned to 180 degrees
- moved C1 13.0 mm to (127.0, 104.1), turned to 0 degrees
Connections:
- A1 pad 14: (no net) -> /DRV_SLP
- A1 pad 15: (no net) -> /DRV_STP
- A1 pad 16: (no net) -> /DRV_DIR
- A1 pad 9: (no net) -> /DRV_EN
- J2 pad 1: Net-(A1-Pad3) -> Net-(A1-Pad6)
- J2 pad 2: Net-(A1-Pad4) -> Net-(A1-Pad5)
- J2 pad 3: Net-(A1-Pad5) -> Net-(A1-Pad4)
- J2 pad 4: Net-(A1-Pad6) -> Net-(A1-Pad3)
- J3 pad 11: (no net) -> /LED_MOVING
- J3 pad 13: (no net) -> /LED_OPEN
- J3 pad 15: (no net) -> /LED_CLOSED
- J3 pad 16: (no net) -> /OUT_SESAME_OPENING
- J3 pad 18: (no net) -> /OUT_SESAME_CLOSING
- J3 pad 22: (no net) -> /OUT_SESAME_OPEN
- J3 pad 26: (no net) -> /IN_KEY
- J3 pad 29: (no net) -> /DRV_SLP
- J3 pad 31: (no net) -> /DRV_EN
- J3 pad 33: (no net) -> /DRV_STP
- J3 pad 35: (no net) -> /DRV_DIR
- J3 pad 36: (no net) -> /IN_MWC
- J3 pad 38: (no net) -> /IN_MWO
- J3 pad 40: (no net) -> /IN_WIN
Routing:
- net GND: track 0.00 -> 121.6 mm
- net /P12V: track 0.00 -> 63.3 mm
- net /P3V3: track 31.3 -> 79.1 mm
- net Net-(D2-Pad1): track 0.00 -> 28.1 mm
- net Net-(D3-Pad1): track 0.00 -> 13.6 mm
- net Net-(A1-Pad3): track 0.00 -> 11.5 mm
- net Net-(A1-Pad4): track 0.00 -> 11.5 mm
- net Net-(A1-Pad5): track 0.00 -> 11.4 mm
- net Net-(A1-Pad6): track 0.00 -> 11.4 mm
- net Net-(D1-Pad1): track 0.00 -> 5.96 mm
- net Net-(J9-Pad2): track 9.58 -> 6.91 mm
- net (no net): vias 0 -> 3
- removed copper zone on F.Cu, net GND
- removed copper zone on In2.Cu, net GND
Other:
- board text added: "CLOSED"
- board text added: "MOVING"
- board text added: "OPEN"

Commit message: finished pcb layout
Parts:
- added REF**: OSHW-Logo2_9.8x8mm_SilkScreen, Symbol:OSHW-Logo2_9.8x8mm_SilkScreen, B.Cu at (83.5, 80.4)
- R1: value 5K -> 470
- R2: renamed from R3; value 5K -> 1K
- R3: renamed from R2; value 5K -> 680
- moved J11 23.0 mm to (132.2, 110.5)
- moved J10 22.9 mm to (109.2, 110.5)
- moved J15 8.89 mm to (91.4, 110.5)
- moved J8 8.89 mm to (100.3, 110.5)
- moved Q1 5.66 mm to (92.7, 72.1), turned to 0 degrees
- moved J9 0.70 mm to (113.7, 74.8)
Connections:
- J3 pad 1: /P3V3 -> (no net)
- J3 pad 10: (no net) -> /LED_CLOSED
- J3 pad 11: /LED_MOVING -> /IN_KEY
- J3 pad 13: /LED_OPEN -> /IN_MWO
- J3 pad 14: GND -> (no net)
- J3 pad 15: /LED_CLOSED -> /IN_MWC
- J3 pad 16: /OUT_SESAME_OPENING -> (no net)
- J3 pad 17: (no net) -> /P3V3
- J3 pad 18: /OUT_SESAME_CLOSING -> (no net)
- J3 pad 20: GND -> (no net)
- J3 pad 22: /OUT_SESAME_OPEN -> (no net)
- J3 pad 25: GND -> (no net)
- J3 pad 26: /IN_KEY -> (no net)
- J3 pad 29: /DRV_SLP -> /DRV_DIR
- J3 pad 31: /DRV_EN -> (no net)
- J3 pad 32: (no net) -> /DRV_STP
- J3 pad 33: /DRV_STP -> /DRV_SLP
- J3 pad 34: GND -> (no net)
- J3 pad 35: /DRV_DIR -> /DRV_EN
- J3 pad 36: /IN_MWC -> /OUT_SESAME_OPEN
- J3 pad 37: (no net) -> /IN_WIN
- J3 pad 38: /IN_MWO -> /OUT_SESAME_CLOSING
- J3 pad 39: GND -> (no net)
- J3 pad 40: /IN_WIN -> /OUT_SESAME_OPENING
- J3 pad 6: GND -> (no net)
- J3 pad 7: (no net) -> /LED_OPEN
- J3 pad 8: (no net) -> /LED_MOVING
- J3 pad 9: GND -> (no net)
Routing:
- net GND: track 121.6 -> 176.4 mm
- net /IN_MWC: track 0.00 -> 50.2 mm
- net /IN_KEY: track 0.00 -> 49.3 mm
- net /IN_MWO: track 0.00 -> 46.7 mm
- net /IN_WIN: track 0.00 -> 46.5 mm
- net /P3V3: track 79.1 -> 125.0 mm
- net /DRV_STP: track 0.00 -> 35.5 mm
- net /DRV_SLP: track 0.00 -> 32.4 mm
- net /DRV_DIR: track 0.00 -> 31.7 mm
- net /LED_MOVING: track 0.00 -> 23.3 mm, vias 0 -> 1
- net /P5V: track 8.71 -> 31.4 mm
- net /LED_CLOSED: track 0.00 -> 22.3 mm, vias 0 -> 1
- net /DRV_EN: track 0.00 -> 21.5 mm
- net /LED_OPEN: track 0.00 -> 19.7 mm, vias 0 -> 1
- net /OUT_SESAME_OPEN: track 0.00 -> 16.8 mm
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- removed copper zone on B.Cu, net /P3V3
- removed copper zone on F.Cu, net /P5V
- removed copper zone on B.Cu, net /P5V_HAT
Other:
- board text added: "8-28V -(o+"
- board text added: "MOTOR"
- board text added: "SESAME"
- board text added: "SW_KEY"
- board text added: "SW_MWC"
- board text added: "SW_MWO"
