File: Elektronik/Raspberry-Motorsteuerung/raspberrypi_hat.sch (KiCad schematic (older format))
At the start: 35 parts, among them J1 Barrel_Jack_Switch, J10 Conn_01x04_Female, J2 M04JST-PTH, J3 40HAT, J4 Conn_01x04_Female, J5 Conn_01x04_Male, J6 Conn_01x04_Male, J7 Conn_Beeper, J8 Conn_01x04_Male, J9 CONN_01X02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

Commit message: TODO bearbeitet
Other:
- note added: "* ENABLE schaltet nur FETs aus, also immer AN machen, da SLEEP die FETs auch aus macht \n(und noch mehr) (wake up time 1 ms beachten!)\n* LEDs direkt auf Platine (die von außen sichtbar anzubringen ist) (und Platine beschriften)\n* Switches auf 2 polige connectors umstellen (weil unterschiedlich lange kabellängen etc)\n* Beeper Verstärker? (PWM reicht eig)\n* Beeper auch noch unnötig, da Schlüsse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"
- note removed: "* Beeper Verstärker\n* mehr Zahnräder, Lichteffekte und SteamPunk für ne gute Show\n (SESAME_OPENING, SESAME_CLOSING)\n\n\n"

Commit message: finished schema, started pcb
Parts:
- removed J10, J4: Conn_01x04_Female, symbol Connector:Conn_01x04_Female
- removed J2: M04JST-PTH, JST-4-PTH, symbol SparkFun-Connectors:M04JST-PTH
- removed J5, J8: Conn_01x04_Male, symbol Connector:Conn_01x04_Male
- removed J7: Conn_Beeper, symbol Connector:Conn_01x02_Male
- added J10, J11, J15, J8: Conn_01x02_Male, Connector_JST:JST_EH_S2B-EH_1x02_P2.50mm_Horizontal, symbol Connector:Conn_01x02_Male
- added J12, J13, J14, J16: Conn_01x02_Female, symbol Connector:Conn_01x02_Female
- added J2: Conn_01x04_Male, Connector_JST:JST_EH_S4B-EH_1x04_P2.50mm_Horizontal, symbol Connector:Conn_01x04_Male
- added SW4: SW_Key, symbol Switch:SW_Push_Open
- D1, D2, D3: footprint (none) -> LED_THT:LED_D5.0mm
- J6: footprint (none) -> Connector_JST:JST_EH_S4B-EH_1x04_P2.50mm_Horizontal
- R1, R2, R3: value R -> 5K; footprint (none) -> Resistor_SMD:R_0603_1608Metric_Pad0.98x0.95mm_HandSolder
- renumbered SW_MWO1 to SW1, SW_WIN1 to SW2, SW_MWC1 to SW3
Connections:
- net GND: now also D1.2 (A), D2.2 (A), D3.2 (A)
- net IN_MWC: now also J10.2 (Pin_2)
- net IN_MWO: now also J8.2 (Pin_2)
- net IN_WIN: now also J11.2 (Pin_2)
- net LED_CLOSED: now also J3.15 (BCM22); no longer J3.10 (BCM15)
- net LED_MOVING: now also J3.11 (BCM17); no longer J3.12 (BCM18)
- net LED_OPEN: now also J3.13 (BCM27); no longer J3.8 (BCM14)
- net P3V3: now also J10.1 (Pin_1), J11.1 (Pin_1), J15.1 (Pin_1), J8.1 (Pin_1)
- net OUT_SESAME_OPEN: now reaches J3.22 (BCM25)
- net OUT_SESAME_OPEN: now also J6.3 (Pin_3)
- net IN_KEY: now reaches J3.26 (BCM7)
- net IN_KEY: now also J15.2 (Pin_2)
- net at A1.3 (1B): now also J2.4 (Pin_4)
- net at A1.4 (1A): now also J2.3 (Pin_3)
- net at A1.5 (2A): now also J2.2 (Pin_2)
- net at A1.6 (2B): now also J2.1 (Pin_1)
- net at SW1.1 (A): now also J12.2 (Pin_2)
- net at SW3.1 (A): now also J14.2 (Pin_2)
- net at SW2.1: now also J13.2 (Pin_2)
- net at R1.2: now also D1.1 (K)
- net at R2.2: now also D2.1 (K)
- net at R3.2: now also D3.1 (K)
- net OUT_BEEPER: no longer names the net of J3.32 (BCM12)
- new net: J12.1 (Pin_1), SW1.2 (B)
- new net: J14.1 (Pin_1), SW3.2 (B)
- new net: J13.1 (Pin_1), SW2.2
- new net: J16.2 (Pin_2), SW4.1 (A)
- new net: J16.1 (Pin_1), SW4.2 (B)
- no-connect marks 4 -> 3
Other:
- note added: "* ENABLE schaltet nur FETs aus, also immer AN machen, da SLEEP die FETs auch aus macht \n(und noch mehr) (wake up time 1 ms beachten!)\n* LEDs direkt auf Platine (die von außen sichtbar anzubringen ist) (und Platine beschriften)\n* Beeper auch noch unnötig, da Schlüsselschalter fehlt (und im mehrräumigem Lab auch wenig Sinn macht)\n* mehr Zahnräder, Lichteffekte und SteamPunk für ne gute Show\n (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"
- note removed: "* ENABLE schaltet nur FETs aus, also immer AN machen, da SLEEP die FETs auch aus macht \n(und noch mehr) (wake up time 1 ms beachten!)\n* LEDs direkt auf Platine (die von außen sichtbar anzubringen ist) (und Platine beschriften)\n* Switches auf 2 polige connectors umstellen (weil unterschiedlich lange kabellängen etc)\n* Beeper Verstärker? (PWM reicht eig)\n* Beeper auch noch unnötig, da Schlüsse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"
- moved on the sheet: D1, D2, D3, SW2, SW3

Commit message: finished pcb layout
Parts:
- D1: value LED -> LED_RED
- D2: value LED -> LED_GREEN
- D3: value LED -> LED_YELLOW
- R1: value 5K -> 470
- R2: renamed from R3; value 5K -> 1K
- R3: renamed from R2; value 5K -> 680
Connections:
- net DRV_DIR: now also J3.29 (BCM5); no longer J3.35 (BCM19)
- net DRV_EN: now also J3.35 (BCM19); no longer J3.31 (BCM6)
- net DRV_SLP: now also J3.33 (BCM13); no longer J3.29 (BCM5)
- net DRV_STP: now also J3.32 (BCM12); no longer J3.33 (BCM13)
- net GND: no longer J3.14 (GND), J3.20 (GND), J3.25 (GND), J3.34 (GND), J3.39 (GND), J3.6 (GND), J3.9 (GND)
- net IN_KEY: now also J3.11 (BCM17); no longer J3.26 (BCM7)
- net IN_MWC: now also J3.15 (BCM22); no longer J3.36 (BCM16)
- net IN_MWO: now also J3.13 (BCM27); no longer J3.38 (BCM20)
- net IN_WIN: now also J3.37 (BCM26); no longer J3.40 (BCM21)
- net LED_CLOSED: now also J3.10 (BCM15); no longer J3.15 (BCM22)
- net LED_MOVING: now also J3.8 (BCM14); no longer J3.11 (BCM17)
- net LED_OPEN: now also J3.7 (BCM4); no longer J3.13 (BCM27)
- net OUT_SESAME_CLOSING: now also J3.38 (BCM20); no longer J3.18 (BCM24)
- net OUT_SESAME_OPEN: now also J3.36 (BCM16); no longer J3.22 (BCM25)
- net OUT_SESAME_OPENING: now also J3.40 (BCM21); no longer J3.16 (BCM23)
- net P3V3: now also J3.17 (P3V3); no longer J3.1 (P3V3)
- no-connect marks 3 -> 23
Other:
- note added: "Zukunftsmusik"
- moved on the sheet: D1, D2, D3, J6, R1, R2, R3
Changed lines of the file:
@@
 Text Notes 1650 2000 0    118  ~ 24
 40-Pin HAT Connector
-Text Label 800  4150 0    60   ~ 0
-GND
-Wire Wire Line
-	2000 4150 800  4150
 Text Label 800  3550 0    60   ~ 0
 ID_SD_EEPROM
 Wire Wire Line
 	2000 3550 800  3550
-Text Label 800  3450 0    60   ~ 0
-GND
-Wire Wire Line
-	2000 3450 800  3450
-Text Label 800  2650 0    60   ~ 0
-GND
-Wire Wire Line
-	2000 2650 800  2650
-Text Label 800  2250 0    60   ~ 0
-P3V3
-Wire Wire Line
-	2000 2250 800  2250
-Wire Wire Line
-	3200 2850 4400 2850
-Wire Wire Line
-	3200 3150 4400 3150
 Wire Wire Line
 	3200 3550 4400 3550
 Wire Wire Line
 	3200 3650 4400 3650
-Wire Wire Line
-	3200 3850 4400 3850
-Text Label 4400 2850 2    60   ~ 0
-GND
-Text Label 4400 3150 2    60   ~ 0
-GND
 Text Label 4400 3650 2    60   ~ 0
 GND
 Text Label 4400 3550 2    60   ~ 0
 ID_SC_EEPROM
-Text Label 4400 3850 2    60   ~ 0
-GND
-Text Label 4400 2450 2    60   ~ 0
-GND
-Wire Wire Line
-	3200 2450 4400 2450
 Text Label 4400 2350 2    60   ~ 0
 P5V_HAT
@@
 Text Label 7800 7150 0    50   ~ 0
 DRV_SLP
-Text Label 800  3650 0    50   ~ 0
+Text Label 800  3850 0    50   ~ 0
 DRV_SLP
-Text Label 800  3750 0    50   ~ 0
-DRV_EN
 Text Label 800  3950 0    50   ~ 0
+DRV_EN
+Text Label 800  3650 0    50   ~ 0
 DRV_DIR
-Text Label 800  3850 0    50   ~ 0
+Text Label 4400 3750 2    50   ~ 0
 DRV_STP
 Wire Wire Line
 	800  3650 2000 3650
 Wire Wire Line
-	800  3750 2000 3750
-Wire Wire Line
 	800  3850 2000 3850
 Wire Wire Line
@@
 Text Label 10650 7900 0    50   ~ 0
 IN_WIN
-Text Label 4400 3950 2    50   ~ 0
-IN_MWC
-Text Label 4400 4050 2    50   ~ 0
-IN_MWO
-Text Label 4400 4150 2    50   ~ 0
+Text Label 800  4050 0    50   ~ 0
 IN_WIN
 Wire Wire Line
@@
 L pspice:R R1
 U 1 1 5FE9D008
-P 6200 7950
-F 0 "R1" V 5995 7950 50  0000 C CNN
-F 1 "5K" V 6086 7950 50  0000 C CNN
-F 2 "Resistor_SMD:R_0603_1608Metric_Pad0.98x0.95mm_HandSolder" H 6200 7950 50  0001 C CNN
-F 3 "~" H 6200 7950 50  0001 C CNN
-	1    6200 7950
+P 6200 7600
+F 0 "R1" V 5995 7600 50  0000 C CNN
+F 1 "470" V 6086 7600 50  0000 C CNN
+F 2 "Resistor_SMD:R_0603_1608Metric_Pad0.98x0.95mm_HandSolder" H 6200 7600 50  0001 C CNN
+F 3 "~" H 6200 7600 50  0001 C CNN
+	1    6200 7600
 	0    1    1    0
 $EndComp
 $Comp
-L pspice:R R2
+L pspice:R R3
 U 1 1 5FE9ECF4
-P 6200 8050
-F 0 "R2" V 5995 8050 50  0000 C CNN
-F 1 "5K" V 6086 8050 50  0000 C CNN
-F 2 "Resistor_SMD:R_0603_1608Metric_Pad0.98x0.95mm_HandSolder" H 6200 8050 50  0001 C CNN
-F 3 "~" H 6200 8050 50  0001 C CNN
-	1    6200 8050
+P 6200 8200
+F 0 "R3" V 5995 8200 50  0000 C CNN
+F 1 "680" V 6086 8200 50  0000 C CNN
+F 2 "Resistor_SMD:R_0603_1608Metric_Pad0.98x0.95mm_HandSolder" H 6200 8200 50  0001 C CNN
+F 3 "~" H 6200 8200 50  0001 C CNN
+	1    6200 8200
 	0    1    1    0
 $EndComp
 $Comp
-L pspice:R R3
+L pspice:R R2
 U 1 1 5FE9F166
-P 6200 8150
-F 0 "R3" V 5995 8150 50  0000 C CNN
-F 1 "5K" V 6086 8150 50  0000 C CNN
-F 2 "Resistor_SMD:R_0603_1608Metric_Pad0.98x0.95mm_HandSolder" H 6200 8150 50  0001 C CNN
-F 3 "~" H 6200 8150 50  0001 C CNN
-	1    6200 8150
+P 6200 7900
+F 0 "R2" V 5995 7900 50  0000 C CNN
+F 1 "1K" V 6086 7900 50  0000 C CNN
+F 2 "Resistor_SMD:R_0603_1608Metric_Pad0.98x0.95mm_HandSolder" H 6200 7900 50  0001 C CNN
+F 3 "~" H 6200 7900 50  0001 C CNN
+	1    6200 7900
 	0    1    1    0
 $EndComp
@@
 L power:GND #PWR0105
 U 1 1 5FE9FB7E
-P 6650 8250
-F 0 "#PWR0105" H 6650 8000 50  0001 C CNN
-F 1 "GND" V 6655 8122 50  0000 R CNN
-F 2 "" H 6650 8250 50  0001 C CNN
-F 3 "" H 6650 8250 50  0001 C CNN
-	1    6650 8250
+P 6650 8300
+F 0 "#PWR0105" H 6650 8050 50  0001 C CNN
+F 1 "GND" V 6655 8172 50  0000 R CNN
+F 2 "" H 6650 8300 50  0001 C CNN
+F 3 "" H 6650 8300 50  0001 C CNN
+	1    6650 8300
 	0    -1   -1   0
 $EndComp
-Text Label 6950 7950 2    50   ~ 0
+Text Label 6950 7600 2    50   ~ 0
 LED_OPEN
-Text Label 6950 8050 2    50   ~ 0
+Text Label 6950 8200 2    50   ~ 0
 LED_CLOSED
-Text Label 6950 8150 2    50   ~ 0
+Text Label 6950 7900 2    50   ~ 0
 LED_MOVING
 Wire Wire Line
-	6950 8150 6450 8150
+	6950 7900 6450 7900
 Wire Wire Line
-	6450 8050 6950 8050
+	6450 8200 6950 8200
 Wire Wire Line
-	6950 7950 6450 7950
-Text Label 800  2850 0    50   ~ 0
+	6950 7600 6450 7600
+Text Label 800  2550 0    50   ~ 0
 LED_OPEN
-Text Label 800  2950 0    50   ~ 0
+Text Label 4400 2650 2    50   ~ 0
 LED_CLOSED
-Text Label 800  2750 0    50   ~ 0
+Text Label 4400 2550 2    50   ~ 0
 LED_MOVING
 Wire Wire Line
-	4400 2750 3200 2750
-Wire Wire Line
 	3200 2650 4400 2650
 Wire Wire Line
@@
 L Device:LED D1
 U 1 1 5FF4B1A2
-P 5800 7950
-F 0 "D1" H 5793 7695 50  0000 C CNN
-F 1 "LED" H 5793 7786 50  0000 C CNN
-F 2 "LED_THT:LED_D5.0mm" H 5800 7950 50  0001 C CNN
-F 3 "~" H 5800 7950 50  0001 C CNN
-	1    5800 7950
+P 5800 7600
+F 0 "D1" H 5800 7400 50  0000 C CNN
+F 1 "LED_RED" H 5800 7500 50  0000 C CNN
+F 2 "LED_THT:LED_D5.0mm" H 5800 7600 50  0001 C CNN
+F 3 "~" H 5800 7600 50  0001 C CNN
+	1    5800 7600
 	-1   0    0    1
 $EndComp
@@
 L Device:LED D2
 U 1 1 5FF4BA2C
-P 5800 8050
-F 0 "D2" H 5793 7795 50  0000 C CNN
-F 1 "LED" H 5793 7886 50  0000 C CNN
-F 2 "LED_THT:LED_D5.0mm" H 5800 8050 50  0001 C CNN
-F 3 "~" H 5800 8050 50  0001 C CNN
-	1    5800 8050
+P 5800 8200
+F 0 "D2" H 5800 8000 50  0000 C CNN
+F 1 "LED_GREEN" H 5800 8100 50  0000 C CNN
+F 2 "LED_THT:LED_D5.0mm" H 5800 8200 50  0001 C CNN
+F 3 "~" H 5800 8200 50  0001 C CNN
+	1    5800 8200
 	-1   0    0    1
 $EndComp
@@
 L Device:LED D3
 U 1 1 5FF4C04A
-P 5800 8150
-F 0 "D3" H 5793 7895 50  0000 C CNN
-F 1 "LED" H 5793 7986 50  0000 C CNN
-F 2 "LED_THT:LED_D5.0mm" H 5800 8150 50  0001 C CNN
-F 3 "~" H 5800 8150 50  0001 C CNN
-	1    5800 8150
+P 5800 7900
+F 0 "D3" H 5800 7700 50  0000 C CNN
+F 1 "LED_YELLOW" H 5800 7800 50  0000 C CNN
+F 2 "LED_THT:LED_D5.0mm" H 5800 7900 50  0001 C CNN
+F 3 "~" H 5800 7900 50  0001 C CNN
+	1    5800 7900
 	-1   0    0    1
 $EndComp
 Wire Wire Line
-	5650 7950 5650 8050
-Wire Wire Line
-	5650 8050 5650 8150
-Connection ~ 5650 8050
-Wire Wire Line
-	5650 8150 5650 8250
+	5650 8200 5650 8300
 Wire Wire Line
-	5650 8250 6650 8250
-Connection ~ 5650 8150
+	5650 8300 6650 8300
 Text Notes 6150 6100 2    59   ~ 12
 Power Supply
 Text Notes 8400 6100 2    59   ~ 12
 Motor Driver\n
-Text Notes 5850 7500 2    59   ~ 12
+Text Notes 5650 7350 2    59   ~ 12
 Status
 Text Notes 8500 9000 2    59   ~ 12
 TODO\n
-Text Label 4400 2950 2    60   ~ 0
-OUT_SESAME_OPENING
-Text Label 4400 3050 2    59   ~ 0
-OUT_SESAME_CLOSING
-Wire Wire Line
-	4400 3050 3200 3050
-Wire Wire Line
-	3200 2950 4400 2950
 $Comp
 L Connector:Conn_01x04_Male J6
 U 1 1 5FFC569D
-P 5750 8650
-F 0 "J6" H 5750 8900 50  0000 C CNN
-F 1 "Conn_01x04_Male" H 5858 8840 50  0001 C CNN
-F 2 "Connector_JST:JST_EH_S4B-EH_1x04_P2.50mm_Horizontal" H 5750 8650 50  0001 C CNN
-F 3 "~" H 5750 8650 50  0001 C CNN
-	1    5750 8650
+P 5700 9000
+F 0 "J6" H 5700 9250 50  0000 C CNN
+F 1 "Conn_01x04_Male" H 5808 9190 50  0001 C CNN
+F 2 "Connector_JST:JST_EH_S4B-EH_1x04_P2.50mm_Horizontal" H 5700 9000 50  0001 C CNN
+F 3 "~" H 5700 9000 50  0001 C CNN
+	1    5700 9000
 	1    0    0    -1
 $EndComp
@@
 L power:GND #PWR0106
 U 1 1 5FFC72D4
-P 5950 8850
-F 0 "#PWR0106" H 5950 8600 50  0001 C CNN
-F 1 "GND" V 5955 8722 50  0000 R CNN
-F 2 "" H 5950 8850 50  0001 C CNN
-F 3 "" H 5950 8850 50  0001 C CNN
-	1    5950 8850
+P 5900 9200
+F 0 "#PWR0106" H 5900 8950 50  0001 C CNN
+F 1 "GND" V 5905 9072 50  0000 R CNN
+F 2 "" H 5900 9200 50  0001 C CNN
+F 3 "" H 5900 9200 50  0001 C CNN
+	1    5900 9200
 	0    -1   -1   0
 $EndComp
-Text Label 6850 8550 2    50   ~ 0
+Text Label 6800 8900 2    50   ~ 0
 OUT_SESAME_OPENING
-Text Label 6850 8650 2    50   ~ 0
+Text Label 6800 9000 2    50   ~ 0
 OUT_SESAME_CLOSING
 Wire Wire Line
-	6850 8550 5950 8550
+	6800 8900 5900 8900
 Wire Wire Line
-	6850 8650 5950 8650
+	6800 9000 5900 9000
 $Bitmap
 Pos 12700 3000
@@
 Wire Wire Line
 	10650 8300 11150 8300
-Text Label 4350 3450 2    50   ~ 0
+Text Label 800  2750 0    50   ~ 0
 IN_KEY
-Text Label 6850 8750 2    50   ~ 0
-OUT_SESAME_OPEN
-Wire Wire Line
-	6850 8750 5950 8750
-Text Label 4400 3250 2    50   ~ 0
+Text Label 6800 9100 2    50   ~ 0
 OUT_SESAME_OPEN
 Wire Wire Line
-	4400 3250 3200 3250
-Wire Wire Line
-	4350 3450 3200 3450
+	6800 9100 5900 9100
 $Comp
 L Connector:Conn_01x04_Male J2
@@
 Wire Wire Line
 	2000 2950 800  2950
+Text Label 800  3050 0    60   ~ 0
+P3V3
+Wire Wire Line
+	2000 3050 800  3050
+Text Label 800  2850 0    50   ~ 0
+IN_MWO
+Text Label 800  2950 0    50   ~ 0
+IN_MWC
+Text Label 4400 3950 2    50   ~ 0
+OUT_SESAME_OPEN
+Text Label 4400 4050 2    59   ~ 0
+OUT_SESAME_CLOSING
+Text Label 4400 4150 2    60   ~ 0
+OUT_SESAME_OPENING
+Wire Wire Line
+	4400 3750 3200 3750
+Wire Wire Line
+	800  4050 2000 4050
+Wire Wire Line
+	800  2550 2000 2550
+NoConn ~ 2000 2350
+NoConn ~ 2000 2450
+NoConn ~ 2000 3150
+NoConn ~ 2000 3250
+NoConn ~ 2000 3350
+NoConn ~ 3200 3350
+NoConn ~ 2000 3450
+NoConn ~ 2000 4150
+NoConn ~ 3200 3850
+NoConn ~ 3200 2750
+NoConn ~ 3200 2450
+NoConn ~ 2000 2650
+NoConn ~ 3200 2850
+NoConn ~ 3200 2950
+NoConn ~ 3200 3050
+NoConn ~ 3200 3150
+NoConn ~ 3200 3250
+NoConn ~ 3200 3450
+NoConn ~ 2000 3750
+NoConn ~ 2000 2250
+Wire Wire Line
+	5650 7600 5650 7900
+Connection ~ 5650 7900
+Connection ~ 5650 8200
+Wire Wire Line
+	5650 7900 5650 8200
+Text Notes 5450 8700 0    59   ~ 12
+Zukunftsmusik
 $EndSCHEMATC

Commit message: improved barrel-jack/capacitor footprint and 12v lanes
Parts:
- C1: footprint SparkFun-Capacitors:CPOL-RADIAL-100UF-25V -> Capacitor_THT:CP_Radial_D6.3mm_P2.50mm
- J1: footprint SparkFun-Connectors:POWER_JACK_PTH_BREAD -> Connector_BarrelJack:BarrelJack_Wuerth_6941xx301002
Changed lines of the file:
@@
 F 0 "J1" H 5407 6867 50  0000 C CNN
 F 1 "Barrel_Jack_Switch" H 5407 6776 50  0000 C CNN
-F 2 "SparkFun-Connectors:POWER_JACK_PTH_BREAD" H 5400 6510 50  0001 C CNN
+F 2 "Connector_BarrelJack:BarrelJack_Wuerth_6941xx301002" H 5400 6510 50  0001 C CNN
 F 3 "~" H 5400 6510 50  0001 C CNN
 	1    5350 6550
@@
 F 0 "C1" V 9615 6500 50  0000 C CNN
 F 1 "100UF-63V-20%_ELECT_" V 9524 6500 50  0000 C CNN
-F 2 "SparkFun-Capacitors:CPOL-RADIAL-100UF-25V" H 9380 6700 20  0001 C CNN
+F 2 "Capacitor_THT:CP_Radial_D6.3mm_P2.50mm" H 9380 6700 20  0001 C CNN
 F 3 "" H 9350 6550 50  0001 C CNN
 	1    9350 6550

Commit message: fixed LED orientation, C1 symbol, added 'rev 2' label, did not export gerber files
Parts:
- C1: symbol SparkFun-Capacitors:100UF-63V-20%_ELECT_ -> Device:CP
Connections:
- net GND: now also C1.2, D1.1 (K), D2.1 (K), D3.1 (K); no longer C1.-, D1.2 (A), D2.2 (A), D3.2 (A)
- net P12V: now also C1.1; no longer C1.+
- net at R1.2: now also D1.2 (A); no longer D1.1 (K)
- net at R3.2: now also D2.2 (A); no longer D2.1 (K)
- net at R2.2: now also D3.2 (A); no longer D3.1 (K)
Other:
- moved on the sheet: D1, D2, D3
Changed lines of the file:
@@
 	8600 6550 8600 6750
 $Comp
-L SparkFun-Capacitors:100UF-63V-20%_ELECT_ C1
-U 1 1 5FE44D33
-P 9350 6550
-F 0 "C1" V 9615 6500 50  0000 C CNN
-F 1 "100UF-63V-20%_ELECT_" V 9524 6500 50  0000 C CNN
-F 2 "Capacitor_THT:CP_Radial_D6.3mm_P2.50mm" H 9380 6700 20  0001 C CNN
-F 3 "" H 9350 6550 50  0001 C CNN
-	1    9350 6550
-	0    -1   -1   0
-$EndComp
-$Comp
 L power:GND #PWR06
 U 1 1 5FE47CF1
@@
 U 1 1 5FF4B1A2
 P 5800 7600
-F 0 "D1" H 5800 7400 50  0000 C CNN
-F 1 "LED_RED" H 5800 7500 50  0000 C CNN
+F 0 "D1" H 5800 7500 50  0000 C CNN
+F 1 "LED_RED" H 5800 7700 50  0000 C CNN
 F 2 "LED_THT:LED_D5.0mm" H 5800 7600 50  0001 C CNN
 F 3 "~" H 5800 7600 50  0001 C CNN
 	1    5800 7600
-	-1   0    0    1
+	1    0    0    -1
 $EndComp
 $Comp
@@
 U 1 1 5FF4BA2C
 P 5800 8200
-F 0 "D2" H 5800 8000 50  0000 C CNN
-F 1 "LED_GREEN" H 5800 8100 50  0000 C CNN
+F 0 "D2" H 5800 8050 50  0000 C CNN
+F 1 "LED_GREEN" H 5775 8300 50  0000 C CNN
 F 2 "LED_THT:LED_D5.0mm" H 5800 8200 50  0001 C CNN
 F 3 "~" H 5800 8200 50  0001 C CNN
 	1    5800 8200
-	-1   0    0    1
+	1    0    0    -1
 $EndComp
 $Comp
@@
 U 1 1 5FF4C04A
 P 5800 7900
-F 0 "D3" H 5800 7700 50  0000 C CNN
-F 1 "LED_YELLOW" H 5800 7800 50  0000 C CNN
+F 0 "D3" H 5800 7800 50  0000 C CNN
+F 1 "LED_YELLOW" H 5800 8000 50  0000 C CNN
 F 2 "LED_THT:LED_D5.0mm" H 5800 7900 50  0001 C CNN
 F 3 "~" H 5800 7900 50  0001 C CNN
 	1    5800 7900
-	-1   0    0    1
+	1    0    0    -1
 $EndComp
 Wire Wire Line
-	5650 8200 5650 8300
-Wire Wire Line
 	5650 8300 6650 8300
 Text Notes 6150 6100 2    59   ~ 12
@@
 NoConn ~ 2000 3750
 NoConn ~ 2000 2250
-Wire Wire Line
-	5650 7600 5650 7900
-Connection ~ 5650 7900
-Connection ~ 5650 8200
-Wire Wire Line
-	5650 7900 5650 8200
 Text Notes 5450 8700 0    59   ~ 12
 Zukunftsmusik
@@
 	-1   0    0    1
 $EndComp
+Wire Wire Line
+	5650 7600 5650 7900
+Connection ~ 5650 7900
+Wire Wire Line
+	5650 7900 5650 8200
+Connection ~ 5650 8200
+Wire Wire Line
+	5650 8200 5650 8300
+$Comp
+L Device:CP C1
+U 1 1 5FE44D33
+P 9400 6550
+F 0 "C1" V 9665 6500 50  0000 C CNN
+F 1 "100UF-63V-20%_ELECT_" V 9574 6500 50  0000 C CNN
+F 2 "Capacitor_THT:CP_Radial_D6.3mm_P2.50mm" H 9430 6700 20  0001 C CNN
+F 3 "" H 9400 6550 50  0001 C CNN
+	1    9400 6550
+	0    -1   -1   0
+$EndComp
 $EndSCHEMATC
